Commit message: add urdf and xacro examples

File: rospy_ws04_simulation/src/urdf_basic_test/urdf/xacro/xacro_test.urdf.xacro (robot description, xacro)
@@ -7,4 +7,7 @@
     <xacro:property name="base2ground_hight" value="0.015" />
     <xacro:property name="base_link_z" value="${base2ground_hight + base_link_l / 2 }" />
+    <material name="black">
+        <color rgba="0.0 0.0 0.0 1.0"/>
+    </material>
     <!-- 设置原点 -->
     <link name="base_footprint">
@@ -44,7 +47,5 @@
                 </geometry>
                 <origin xyz="0.0 0.0 0.0" rpy="${pi / 2} 0.0 0.0"/>
-                <material name="black">
-                    <color rgba="0.0 0.0 0.0 1.0"/>
-                </material>
+                <material name="black"/>
             </visual>
         </link>
@@ -67,7 +68,5 @@
                 </geometry>
                 <origin xyz="0.0 0.0 0.0" rpy="0.0 0.0 0.0"/>
-                <material name="black">
-                    <color rgba="0.0 0.0 0.0 1.0"/>
-                </material>
+                <material name="black"/>
             </visual>
         </link>
