Commit message: add gazebo-based moving control, lasar, camera and kinect simulation

File: rospy_ws04_simulation/src/gazebo_test/urdf/xacro/base.urdf.xacro (robot description, xacro)
@@ -72,7 +72,5 @@
         </link>
         <gazebo reference="${name}_MoveWheel">
-            <material>
-                Gazebo/Red
-            </material>
+            <material>Gazebo/Red</material>
         </gazebo>
         <joint name="${name}_MoveWheel2base_link" type="continuous">
@@ -106,7 +104,5 @@
         </link>
         <gazebo reference="${name}_SupportWheel">
-            <material>
-                Gazebo/Red
-            </material>
+            <material>Gazebo/Red</material>
         </gazebo>
         <joint name="${name}_SupportWheel2base_link" type="continuous">

File: rospy_ws04_simulation/src/gazebo_test/urdf/xacro/comba.urdf.xacro (robot description, xacro)
@@ -4,3 +4,5 @@
     <xacro:include filename="camera.urdf.xacro"/>
     <xacro:include filename="ladar.urdf.xacro"/>
+    <xacro:include filename="move_controller.urdf.xacro"/>
+    <xacro:include filename="sensor_config.urdf.xacro"/>
 </robot>
